Commit message: paolo: update

File: urdf/crx.ros2_control.xacro (robot description, xacro)
@@ -1,10 +1,14 @@
 <?xml version="1.0"?>
 <robot xmlns:xacro="http://www.ros.org/wiki/xacro">
-  <xacro:macro name="crx20_ros2_control" params="name">
+  <xacro:macro name="crx_ros2_control" params="name use_mock_hardware:=false">
     <ros2_control name="${name}" type="system">
       <hardware>
-        <!-- <plugin>mock_components/GenericSystem</plugin> -->
-        <!-- <param name="position_state_following_offset">0.1</param> -->
-        <plugin>fanuc/FanucTopic</plugin>
+        <xacro:if value="${use_mock_hardware}">
+          <plugin>mock_components/GenericSystem</plugin>
+          <!-- <param name="position_state_following_offset">0.1</param> -->
+        </xacro:if>
+        <xacro:unless value="${use_mock_hardware}">
+          <plugin>fanuc/FanucTopic</plugin>
+        </xacro:unless>
       </hardware>
       <joint name="J1">

File: urdf/crx10ia/crx10ia.urdf.xacro (robot description, xacro)
@@ -1,7 +1,8 @@
 <?xml version="1.0"?>
 <robot xmlns:xacro="http://wiki.ros.org/xacro">
-  <xacro:include filename="$(find crx_description)/crx20/urdf/crx20ia_l.ros2_control.xacro"/>
-  <xacro:crx20_ros2_control name="crx20"/>
-  <xacro:macro name="crx20ia_l">
+  <xacro:macro name="crx10ia" params="use_mock_hardware:=false">
+  <xacro:arg name="use_mock_hardware" default="false"/>
+  <xacro:include filename="$(find crx_description)/urdf/crx.ros2_control.xacro"/>
+  <xacro:crx_ros2_control name="crx10" use_mock_hardware="$(arg use_mock_hardware)"/>
     <material name="FANUC_Black">
       <color rgba="0 0 0 1.0"/>
@@ -18,24 +19,24 @@
     <xacro:property name="l_base" value="0.245"/>
     <xacro:property name="l_1" value="0.0"/>
-    <xacro:property name="l_2" value="0.710"/>
+    <xacro:property name="l_2" value="0.540"/>
     <xacro:property name="l_3" value="0.0"/>
     <xacro:property name="l_4" value="0.540"/>
     <xacro:property name="l_5" value="0.150"/>
     <xacro:property name="l_6" value="0.160"/>
-    <xacro:property name="j1_v" value="80"/>
-    <xacro:property name="j2_v" value="80"/>
-    <xacro:property name="j3_v" value="120"/>
-    <xacro:property name="j4_v" value="112.5"/>
-    <xacro:property name="j5_v" value="90"/>
-    <xacro:property name="j6_v" value="112.5"/>
-    <xacro:property name="j1_u" value="179.9"/>
+    <xacro:property name="j1_v" value="120"/>
+    <xacro:property name="j2_v" value="120"/>
+    <xacro:property name="j3_v" value="180"/>
+    <xacro:property name="j4_v" value="180"/>
+    <xacro:property name="j5_v" value="180"/>
+    <xacro:property name="j6_v" value="180"/>
+    <xacro:property name="j1_u" value="190"/>
     <xacro:property name="j2_u" value="179.9"/>
-    <xacro:property name="j3_u" value="270"/>
+    <xacro:property name="j3_u" value="251"/>
     <xacro:property name="j4_u" value="190"/>
     <xacro:property name="j5_u" value="179.9"/>
     <xacro:property name="j6_u" value="225"/>
-    <xacro:property name="j1_l" value="-179.9"/>
+    <xacro:property name="j1_l" value="-190"/>
     <xacro:property name="j2_l" value="-179.9"/>
-    <xacro:property name="j3_l" value="-270"/>
+    <xacro:property name="j3_l" value="-71"/>
     <xacro:property name="j4_l" value="-190"/>
     <xacro:property name="j5_l" value="-179.9"/>
@@ -43,5 +44,5 @@
     <xacro:property name="mz_1" value="0.1277"/>
     <xacro:property name="mz_2" value="0.245"/>
-    <xacro:property name="mz_3" value="0.955"/>
+    <xacro:property name="mz_3" value="0.785"/>
     <xacro:property name="mx_1" value="0.540"/>
     <xacro:property name="mx_2" value="0.700"/>
@@ -52,5 +53,5 @@
 	<origin xyz="0 0 0" rpy="0 0 0"/>
 	<geometry>
-	  <mesh filename="package://crx_description/crx20//meshes/crx20ia_l/visual/base.stl" scale="0.001 0.001 0.001"/>
+	  <mesh filename="package://crx_description/meshes/crx10ia/visual/base.stl" scale="0.001 0.001 0.001"/>
 	</geometry>
 	<material name="FANUC_Black"/>
@@ -59,5 +60,5 @@
 	<origin xyz="0 0 0" rpy="0 0 0"/>
 	<geometry>
-	  <mesh filename="package://crx_description/crx20//meshes/crx20ia_l/collision/base.stl" scale="0.001 0.001 0.001"/>
+	  <mesh filename="package://crx_description/meshes/crx10ia/collision/base.stl" scale="0.001 0.001 0.001"/>
 	</geometry>
       </collision>
@@ -67,5 +68,5 @@
         <origin xyz="0 0 ${mz_1 - l_base}" rpy="0 0 0"/>
 	<geometry>
-	  <mesh filename="package://crx_description/crx20//meshes/crx20ia_l/visual/j1.stl" scale="0.001 0.001 0.001"/>
+	  <mesh filename="package://crx_description/meshes/crx10ia/visual/j1.stl" scale="0.001 0.001 0.001"/>
 	</geometry>
 	<material name="FANUC_White"/>
@@ -74,5 +75,5 @@
         <origin xyz="0 0 ${mz_1 - l_base}" rpy="0 0 0"/>
 	<geometry>
-	  <mesh filename="package://crx_description/crx20//meshes/crx20ia_l/collision/j1.stl" scale="0.001 0.001 0.001"/>
+	  <mesh filename="package://crx_description/meshes/crx10ia/collision/j1.stl" scale="0.001 0.001 0.001"/>
 	</geometry>
       </collision>
@@ -82,5 +83,5 @@
         <origin xyz="-${l_1} 0 ${mz_2 - l_base}" rpy="0 0 0"/>
 	<geometry>
-	  <mesh filename="package://crx_description/crx20//meshes/crx20ia_l/visual/j2.stl" scale="0.001 0.001 0.001"/>
+	  <mesh filename="package://crx_description/meshes/crx10ia/visual/j2.stl" scale="0.001 0.001 0.001"/>
 	</geometry>
 	<material name="FANUC_White"/>
@@ -89,5 +90,5 @@
         <origin xyz="-${l_1} 0 ${mz_2 - l_base}" rpy="0 0 0"/>
 	<geometry>
-	  <mesh filename="package://crx_description/crx20//meshes/crx20ia_l/collision/j2.stl" scale="0.001 0.001 0.001"/>
+	  <mesh filename="package://crx_description/meshes/crx10ia/collision/j2.stl" scale="0.001 0.001 0.001"/>
 	</geometry>
       </collision>
@@ -97,5 +98,5 @@
 	<origin xyz="-${l_1} 0 ${mz_3 - l_base - l_2}" rpy="0 0 0"/>
 	<geometry>
-	  <mesh filename="package://crx_description/crx20//meshes/crx20ia_l/visual/j3.stl" scale="0.001 0.001 0.001"/>
+	  <mesh filename="package://crx_description/meshes/crx10ia/visual/j3.stl" scale="0.001 0.001 0.001"/>
 	</geometry>
 	<material name="FANUC_White"/>
@@ -104,5 +105,5 @@
 	<origin xyz="-${l_1} 0 ${mz_3 - l_base - l_2}" rpy="0 0 0"/>
 	<geometry>
-	  <mesh filename="package://crx_description/crx20//meshes/crx20ia_l/collision/j3.stl" scale="0.001 0.001 0.001"/>
+	  <mesh filename="package://crx_description/meshes/crx10ia/collision/j3.stl" scale="0.001 0.001 0.001"/>
 	</geometry>
       </collision>
@@ -112,5 +113,5 @@
 	<origin xyz="${mx_1 - l_1} 0 ${mz_3 - l_base - l_2 - l_3}" rpy="0 0 0"/>
 	<geometry>
-	  <mesh filename="package://crx_description/crx20//meshes/crx20ia_l/visual/j4.stl" scale="0.001 0.001 0.001"/>
+	  <mesh filename="package://crx_description/meshes/crx10ia/visual/j4.stl" scale="0.001 0.001 0.001"/>
 	</geometry>
 	<material name="FANUC_White"/>
@@ -119,5 +120,5 @@
 	<origin xyz="${mx_1 - l_1} 0 ${mz_3 - l_base - l_2 - l_3}" rpy="0 0 0"/>
 	<geometry>
-	  <mesh filename="package://crx_description/crx20//meshes/crx20ia_l/collision/j4.stl" scale="0.001 0.001 0.001"/>
+	  <mesh filename="package://crx_description/meshes/crx10ia/collision/j4.stl" scale="0.001 0.001 0.001"/>
 	</geometry>
       </collision>
@@ -127,5 +128,5 @@
 	<origin xyz="${mx_1 -l_1 - l_4} ${my_1} ${mz_3 - l_base - l_2 - l_3}" rpy="0 0 0"/>
 	<geometry>
-	  <mesh filename="package://crx_description/crx20//meshes/crx20ia_l/visual/j5.stl" scale="0.001 0.001 0.001"/>
+	  <mesh filename="package://crx_description/meshes/crx10ia/visual/j5.stl" scale="0.001 0.001 0.001"/>
 	</geometry>
 	<material name="FANUC_White"/>
@@ -134,5 +135,5 @@
 	<origin xyz="${mx_1 -l_1 - l_4} ${my_1} ${mz_3 - l_base - l_2 - l_3}" rpy="0 0 0"/>
 	<geometry>
-	  <mesh filename="package://crx_description/crx20//meshes/crx20ia_l/collision/j5.stl" scale="0.001 0.001 0.001"/>
+	  <mesh filename="package://crx_description/meshes/crx10ia/collision/j5.stl" scale="0.001 0.001 0.001"/>
 	</geometry>
       </collision>
@@ -142,5 +143,5 @@
 	<origin xyz="${mx_2 -l_1 - l_4} ${my_1 + l_5} ${mz_3 - l_base - l_2 - l_3}" rpy="0 0 0"/>
 	<geometry>
-	  <mesh filename="package://crx_description/crx20//meshes/crx20ia_l/visual/j6.stl" scale="0.001 0.001 0.001"/>
+	  <mesh filename="package://crx_description/meshes/crx10ia/visual/j6.stl" scale="0.001 0.001 0.001"/>
 	</geometry>
 	<material name="FANUC_Black"/>
@@ -149,5 +150,5 @@
 	<origin xyz="${mx_2 -l_1 - l_4} ${my_1 + l_5} ${mz_3 - l_base - l_2 - l_3}" rpy="0 0 0"/>
 	<geometry>
-	  <mesh filename="package://crx_description/crx20//meshes/crx20ia_l/collision/j6.stl" scale="0.001 0.001 0.001"/>
+	  <mesh filename="package://crx_description/meshes/crx10ia/collision/j6.stl" scale="0.001 0.001 0.001"/>
 	</geometry>
       </collision>
@@ -220,5 +221,5 @@
     <link name="tcp" />
     <joint name="flange1-tcp" type="fixed">
-      <origin xyz="0 0 0.18" rpy="0 0 0" />
+      <origin xyz="0 0 0" rpy="0 0 0" />
       <parent link="flange1" />
       <child link="tcp" />

File: urdf/crx20ia_l/crx20ia_l.xacro (robot description, xacro)
@@ -1,5 +1,5 @@
 <?xml version="1.0"?>
 <robot name="crx20ia_l" xmlns:xacro="http://wiki.ros.org/xacro">
-  <xacro:include filename="$(find crx_description)/crx20/urdf/crx20ia_l.urdf.xacro"/>
+  <xacro:include filename="$(find crx_description)/urdf/crx20ia_l/crx20ia_l.urdf.xacro"/>
   <!-- <xacro:include filename="$(find crx_description)/crx20/urdf/crx20ia_l.ros2_control.xacro"/> -->
   <xacro:crx20ia_l/>

Commit message: paolo: ip from command line (crx20 only)

File: urdf/crx.ros2_control.xacro (robot description, xacro)
@@ -1,5 +1,5 @@
 <?xml version="1.0"?>
 <robot xmlns:xacro="http://www.ros.org/wiki/xacro">
-  <xacro:macro name="crx_ros2_control" params="name use_mock_hardware:=false">
+  <xacro:macro name="crx_ros2_control" params="name robot_ip:=10.11.31.111 use_mock_hardware:=false">
     <ros2_control name="${name}" type="system">
       <hardware>
@@ -9,5 +9,6 @@
         </xacro:if>
         <xacro:unless value="${use_mock_hardware}">
-          <plugin>fanuc/FanucTopic</plugin>
+          <plugin>fanuc/FanucHw</plugin>
+          <param name="robot_ip">${robot_ip}</param>
         </xacro:unless>
       </hardware>

File: urdf/crx20ia_l/crx20ia_l.urdf.xacro (robot description, xacro)
@@ -1,8 +1,9 @@
 <?xml version="1.0"?>
 <robot xmlns:xacro="http://wiki.ros.org/xacro">
-  <xacro:macro name="crx20ia_l" params="use_mock_hardware:=false">
+  <xacro:macro name="crx20ia_l" params="robot_ip:=10.11.31.121 use_mock_hardware:=false">
   <xacro:arg name="use_mock_hardware" default="false"/>
+  <xacro:arg name="robot_ip" default="10.11.31.111"/>
   <xacro:include filename="$(find crx_description)/urdf/crx.ros2_control.xacro"/>
-  <xacro:crx_ros2_control name="crx20" use_mock_hardware="$(arg use_mock_hardware)"/>
+  <xacro:crx_ros2_control name="crx20" use_mock_hardware="$(arg use_mock_hardware)" robot_ip="$(arg robot_ip)"/>
     <material name="FANUC_Black">
       <color rgba="0 0 0 1.0"/>

Commit message: paolo: read only available

File: urdf/crx.ros2_control.xacro (robot description, xacro)
@@ -1,5 +1,10 @@
 <?xml version="1.0"?>
 <robot xmlns:xacro="http://www.ros.org/wiki/xacro">
-  <xacro:macro name="crx_ros2_control" params="name robot_ip:=10.11.31.111 use_mock_hardware:=false">
+  <xacro:macro name="crx_ros2_control"
+  params="name
+  robot_ip:=10.11.31.111
+  use_mock_hardware:=false
+  read_only:=false">
+  <!-- Read only parameter should allow to move the robot via manual guidance, jog, etc throu the TP, and makes available the /joint_states topic -->
     <ros2_control name="${name}" type="system">
       <hardware>
@@ -11,4 +16,5 @@
           <plugin>fanuc/FanucHw</plugin>
           <param name="robot_ip">${robot_ip}</param>
+          <param name="read_only">${read_only}</param>
         </xacro:unless>
       </hardware>

File: urdf/crx20ia_l/crx20ia_l.urdf.xacro (robot description, xacro)
@@ -1,9 +1,17 @@
 <?xml version="1.0"?>
 <robot xmlns:xacro="http://wiki.ros.org/xacro">
-  <xacro:macro name="crx20ia_l" params="robot_ip:=10.11.31.121 use_mock_hardware:=false">
+  <xacro:macro name="crx20ia_l"
+  params="robot_ip:=10.11.31.121
+  read_only:=false
+  use_mock_hardware:=false">
   <xacro:arg name="use_mock_hardware" default="false"/>
   <xacro:arg name="robot_ip" default="10.11.31.111"/>
+  <xacro:arg name="read_only" default="false"/>
   <xacro:include filename="$(find crx_description)/urdf/crx.ros2_control.xacro"/>
-  <xacro:crx_ros2_control name="crx20" use_mock_hardware="$(arg use_mock_hardware)" robot_ip="$(arg robot_ip)"/>
+  <xacro:crx_ros2_control
+  name="crx20"
+  use_mock_hardware="$(arg use_mock_hardware)"
+  robot_ip="$(arg robot_ip)"
+  read_only="$(arg read_only)"/>
     <material name="FANUC_Black">
       <color rgba="0 0 0 1.0"/>
