Commit message: paolo: updated crx25 with ip and read opnly parameters. TODO to the others

File: urdf/crx20ia_l/crx20ia_l.urdf.xacro (robot description, xacro)
@@ -2,16 +2,15 @@
 <robot xmlns:xacro="http://wiki.ros.org/xacro">
   <xacro:macro name="crx20ia_l"
-  params="robot_ip:=10.11.31.121
-  read_only:=false
-  use_mock_hardware:=false">
+               params="robot_ip:=10.11.31.121
+               read_only:=false
+               use_mock_hardware:=false">
   <xacro:arg name="use_mock_hardware" default="false"/>
   <xacro:arg name="robot_ip" default="10.11.31.111"/>
   <xacro:arg name="read_only" default="false"/>
   <xacro:include filename="$(find crx_description)/urdf/crx.ros2_control.xacro"/>
-  <xacro:crx_ros2_control
-  name="crx20"
-  use_mock_hardware="$(arg use_mock_hardware)"
-  robot_ip="$(arg robot_ip)"
-  read_only="$(arg read_only)"/>
+  <xacro:crx_ros2_control name="crx20"
+                          use_mock_hardware="$(arg use_mock_hardware)"
+                          robot_ip="$(arg robot_ip)"
+                          read_only="$(arg read_only)"/>
     <material name="FANUC_Black">
       <color rgba="0 0 0 1.0"/>

File: urdf/crx25ia_l/crx25ia_l.urdf.xacro (robot description, xacro)
@@ -1,8 +1,16 @@
 <?xml version="1.0"?>
 <robot xmlns:xacro="http://wiki.ros.org/xacro">
-  <xacro:macro name="crx25ia_l" params="use_mock_hardware:=false">
+  <xacro:macro name="crx25ia_l"
+               params="robot_ip:=10.11.31.121
+               read_only:=false
+               use_mock_hardware:=false">
   <xacro:arg name="use_mock_hardware" default="false"/>
+  <xacro:arg name="robot_ip" default="10.11.31.111"/>
+  <xacro:arg name="read_only" default="false"/>
   <xacro:include filename="$(find crx_description)/urdf/crx.ros2_control.xacro"/>
-  <xacro:crx_ros2_control name="crx25" use_mock_hardware="$(arg use_mock_hardware)"/>
+  <xacro:crx_ros2_control name="crx25"
+                          use_mock_hardware="$(arg use_mock_hardware)"
+                          robot_ip="$(arg robot_ip)"
+                          read_only="$(arg read_only)"/>
     <material name="FANUC_Black">
       <color rgba="0 0 0 1.0"/>
