Commit message: fixed crx10ial demo.launch

File: urdf/crx10ia_l/crx10ia_l.urdf_OLD.xacro (robot description, xacro)
@@ -1,15 +1,8 @@
 <?xml version="1.0"?>
 <robot xmlns:xacro="http://wiki.ros.org/xacro">
-  <xacro:macro name="crx10ia_l"
-               params="robot_ip='10.11.31.121'
-               read_only='false'
-               use_rmi='false'
-               use_mock_hardware=false">
-    <xacro:include filename="$(find crx_description)/urdf/crx.ros2_control.xacro" />
-    <xacro:crx_ros2_control name="crx10"
-                            use_mock_hardware="${use_mock_hardware}"
-                            robot_ip="${robot_ip}"
-                            read_only="${read_only}"
-                            use_rmi="${use_rmi}" />
+  <xacro:macro name="crx10ia_l" params="use_mock_hardware:=false">
+  <xacro:arg name="use_mock_hardware" default="false"/>
+  <xacro:include filename="$(find crx_description)/urdf/crx.ros2_control.xacro"/>
+  <xacro:crx_ros2_control name="crx10" use_mock_hardware="$(arg use_mock_hardware)"/>
     <material name="FANUC_Black">
       <color rgba="0 0 0 1.0"/>
@@ -26,24 +19,24 @@
     <xacro:property name="l_base" value="0.245"/>
     <xacro:property name="l_1" value="0.0"/>
-    <xacro:property name="l_2" value="0.710"/>
+    <xacro:property name="l_2" value="0.540"/>
     <xacro:property name="l_3" value="0.0"/>
     <xacro:property name="l_4" value="0.540"/>
     <xacro:property name="l_5" value="0.150"/>
     <xacro:property name="l_6" value="0.160"/>
-    <xacro:property name="j1_v" value="80"/>
-    <xacro:property name="j2_v" value="80"/>
-    <xacro:property name="j3_v" value="120"/>
-    <xacro:property name="j4_v" value="112.5"/>
-    <xacro:property name="j5_v" value="90"/>
-    <xacro:property name="j6_v" value="112.5"/>
-    <xacro:property name="j1_u" value="179.9"/>
+    <xacro:property name="j1_v" value="120"/>
+    <xacro:property name="j2_v" value="120"/>
+    <xacro:property name="j3_v" value="180"/>
+    <xacro:property name="j4_v" value="180"/>
+    <xacro:property name="j5_v" value="180"/>
+    <xacro:property name="j6_v" value="180"/>
+    <xacro:property name="j1_u" value="190"/>
     <xacro:property name="j2_u" value="179.9"/>
-    <xacro:property name="j3_u" value="270"/>
+    <xacro:property name="j3_u" value="251"/>
     <xacro:property name="j4_u" value="190"/>
     <xacro:property name="j5_u" value="179.9"/>
     <xacro:property name="j6_u" value="225"/>
-    <xacro:property name="j1_l" value="-179.9"/>
+    <xacro:property name="j1_l" value="-190"/>
     <xacro:property name="j2_l" value="-179.9"/>
-    <xacro:property name="j3_l" value="-270"/>
+    <xacro:property name="j3_l" value="-71"/>
     <xacro:property name="j4_l" value="-190"/>
     <xacro:property name="j5_l" value="-179.9"/>
@@ -51,5 +44,5 @@
     <xacro:property name="mz_1" value="0.1277"/>
     <xacro:property name="mz_2" value="0.245"/>
-    <xacro:property name="mz_3" value="0.955"/>
+    <xacro:property name="mz_3" value="0.785"/>
     <xacro:property name="mx_1" value="0.540"/>
     <xacro:property name="mx_2" value="0.700"/>
@@ -58,15 +51,15 @@
     <link name="base_link">
       <visual>
-      	<origin xyz="0 0 0" rpy="0 0 0"/>
-      	<geometry>
-      	  <mesh filename="package://crx_description/meshes/crx10ia_l/visual/base.stl" scale="0.001 0.001 0.001"/>
-      	</geometry>
-      	<material name="FANUC_Black"/>
-      </visual>
-      <collision>
-      	<origin xyz="0 0 0" rpy="0 0 0"/>
-      	<geometry>
-      	  <mesh filename="package://crx_description/meshes/crx10ia_l/collision/base.stl" scale="0.001 0.001 0.001"/>
-      	</geometry>
+	<origin xyz="0 0 0" rpy="0 0 0"/>
+	<geometry>
+	  <mesh filename="package://crx_description/meshes/crx10ia_l/visual/base.stl" scale="0.001 0.001 0.001"/>
+	</geometry>
+	<material name="FANUC_Black"/>
+      </visual>
+      <collision>
+	<origin xyz="0 0 0" rpy="0 0 0"/>
+	<geometry>
+	  <mesh filename="package://crx_description/meshes/crx10ia_l/collision/base.stl" scale="0.001 0.001 0.001"/>
+	</geometry>
       </collision>
     </link>
@@ -74,14 +67,14 @@
       <visual>
         <origin xyz="0 0 ${mz_1 - l_base}" rpy="0 0 0"/>
-      	<geometry>
-          <mesh filename="package://crx_description/meshes/crx10ia_l/visual/j1.stl" scale="0.001 0.001 0.001"/>
-      	</geometry>
-      	<material name="FANUC_White"/>
+	<geometry>
+	  <mesh filename="package://crx_description/meshes/crx10ia_l/visual/j1.stl" scale="0.001 0.001 0.001"/>
+	</geometry>
+	<material name="FANUC_White"/>
       </visual>
       <collision>
         <origin xyz="0 0 ${mz_1 - l_base}" rpy="0 0 0"/>
-      	<geometry>
-          <mesh filename="package://crx_description/meshes/crx10ia_l/collision/j1.stl" scale="0.001 0.001 0.001"/>
-      	</geometry>
+	<geometry>
+	  <mesh filename="package://crx_description/meshes/crx10ia_l/collision/j1.stl" scale="0.001 0.001 0.001"/>
+	</geometry>
       </collision>
     </link>
@@ -89,74 +82,74 @@
       <visual>
         <origin xyz="-${l_1} 0 ${mz_2 - l_base}" rpy="0 0 0"/>
-      	<geometry>
-      	  <mesh filename="package://crx_description/meshes/crx10ia_l/visual/j2.stl" scale="0.001 0.001 0.001"/>
-      	</geometry>
-  	    <material name="FANUC_White"/>
+	<geometry>
+	  <mesh filename="package://crx_description/meshes/crx10ia_l/visual/j2.stl" scale="0.001 0.001 0.001"/>
+	</geometry>
+	<material name="FANUC_White"/>
       </visual>
       <collision>
         <origin xyz="-${l_1} 0 ${mz_2 - l_base}" rpy="0 0 0"/>
-      	<geometry>
-      	  <mesh filename="package://crx_description/meshes/crx10ia_l/collision/j2.stl" scale="0.001 0.001 0.001"/>
-      	</geometry>
+	<geometry>
+	  <mesh filename="package://crx_description/meshes/crx10ia_l/collision/j2.stl" scale="0.001 0.001 0.001"/>
+	</geometry>
       </collision>
     </link>
     <link name="J3_link">
       <visual>
-      	<origin xyz="-${l_1} 0 ${mz_3 - l_base - l_2}" rpy="0 0 0"/>
-      	<geometry>
-      	  <mesh filename="package://crx_description/meshes/crx10ia_l/visual/j3.stl" scale="0.001 0.001 0.001"/>
-  	    </geometry>
-        <material name="FANUC_White"/>
-      </visual>
-      <collision>
-      	<origin xyz="-${l_1} 0 ${mz_3 - l_base - l_2}" rpy="0 0 0"/>
-      	<geometry>
-      	  <mesh filename="package://crx_description/meshes/crx10ia_l/collision/j3.stl" scale="0.001 0.001 0.001"/>
-      	</geometry>
+	<origin xyz="-${l_1} 0 ${mz_3 - l_base - l_2}" rpy="0 0 0"/>
+	<geometry>
+	  <mesh filename="package://crx_description/meshes/crx10ia_l/visual/j3.stl" scale="0.001 0.001 0.001"/>
+	</geometry>
+	<material name="FANUC_White"/>
+      </visual>
+      <collision>
+	<origin xyz="-${l_1} 0 ${mz_3 - l_base - l_2}" rpy="0 0 0"/>
+	<geometry>
+	  <mesh filename="package://crx_description/meshes/crx10ia_l/collision/j3.stl" scale="0.001 0.001 0.001"/>
+	</geometry>
       </collision>
     </link>
     <link name="J4_link">
       <visual>
-      	<origin xyz="${mx_1 - l_1} 0 ${mz_3 - l_base - l_2 - l_3}" rpy="0 0 0"/>
-      	<geometry>
-      	  <mesh filename="package://crx_description/meshes/crx10ia_l/visual/j4.stl" scale="0.001 0.001 0.001"/>
-      	</geometry>
-      	<material name="FANUC_White"/>
-      </visual>
-      <collision>
-      	<origin xyz="${mx_1 - l_1} 0 ${mz_3 - l_base - l_2 - l_3}" rpy="0 0 0"/>
-      	<geometry>
-      	  <mesh filename="package://crx_description/meshes/crx10ia_l/collision/j4.stl" scale="0.001 0.001 0.001"/>
-      	</geometry>
+	<origin xyz="${mx_1 - l_1} 0 ${mz_3 - l_base - l_2 - l_3}" rpy="0 0 0"/>
+	<geometry>
+	  <mesh filename="package://crx_description/meshes/crx10ia_l/visual/j4.stl" scale="0.001 0.001 0.001"/>
+	</geometry>
+	<material name="FANUC_White"/>
+      </visual>
+      <collision>
+	<origin xyz="${mx_1 - l_1} 0 ${mz_3 - l_base - l_2 - l_3}" rpy="0 0 0"/>
+	<geometry>
+	  <mesh filename="package://crx_description/meshes/crx10ia_l/collision/j4.stl" scale="0.001 0.001 0.001"/>
+	</geometry>
       </collision>
     </link>
     <link name="J5_link">
       <visual>
-      	<origin xyz="${mx_1 -l_1 - l_4} ${my_1} ${mz_3 - l_base - l_2 - l_3}" rpy="0 0 0"/>
-      	<geometry>
-      	  <mesh filename="package://crx_description/meshes/crx10ia_l/visual/j5.stl" scale="0.001 0.001 0.001"/>
-      	</geometry>
-      	<material name="FANUC_White"/>
-      </visual>
-      <collision>
-      	<origin xyz="${mx_1 -l_1 - l_4} ${my_1} ${mz_3 - l_base - l_2 - l_3}" rpy="0 0 0"/>
-      	<geometry>
-      	  <mesh filename="package://crx_description/meshes/crx10ia_l/collision/j5.stl" scale="0.001 0.001 0.001"/>
-      	</geometry>
+	<origin xyz="${mx_1 -l_1 - l_4} ${my_1} ${mz_3 - l_base - l_2 - l_3}" rpy="0 0 0"/>
+	<geometry>
+	  <mesh filename="package://crx_description/meshes/crx10ia_l/visual/j5.stl" scale="0.001 0.001 0.001"/>
+	</geometry>
+	<material name="FANUC_White"/>
+      </visual>
+      <collision>
+	<origin xyz="${mx_1 -l_1 - l_4} ${my_1} ${mz_3 - l_base - l_2 - l_3}" rpy="0 0 0"/>
+	<geometry>
+	  <mesh filename="package://crx_description/meshes/crx10ia_l/collision/j5.stl" scale="0.001 0.001 0.001"/>
+	</geometry>
       </collision>
     </link>
     <link name="J6_link">
       <visual>
-	      <origin xyz="${mx_2 -l_1 - l_4} ${my_1 + l_5} ${mz_3 - l_base - l_2 - l_3}" rpy="0 0 0"/>
-        <geometry>
-          <mesh filename="package://crx_description/meshes/crx10ia_l/visual/j6.stl" scale="0.001 0.001 0.001"/>
-        </geometry>
-        <material name="FANUC_Black"/>
-      </visual>
-      <collision>
-        <origin xyz="${mx_2 -l_1 - l_4} ${my_1 + l_5} ${mz_3 - l_base - l_2 - l_3}" rpy="0 0 0"/>
-        <geometry>
-          <mesh filename="package://crx_description/meshes/crx10ia_l/collision/j6.stl" scale="0.001 0.001 0.001"/>
-        </geometry>
+	<origin xyz="${mx_2 -l_1 - l_4} ${my_1 + l_5} ${mz_3 - l_base - l_2 - l_3}" rpy="0 0 0"/>
+	<geometry>
+	  <mesh filename="package://crx_description/meshes/crx10ia_l/visual/j6.stl" scale="0.001 0.001 0.001"/>
+	</geometry>
+	<material name="FANUC_Black"/>
+      </visual>
+      <collision>
+	<origin xyz="${mx_2 -l_1 - l_4} ${my_1 + l_5} ${mz_3 - l_base - l_2 - l_3}" rpy="0 0 0"/>
+	<geometry>
+	  <mesh filename="package://crx_description/meshes/crx10ia_l/collision/j6.stl" scale="0.001 0.001 0.001"/>
+	</geometry>
       </collision>
     </link>

File: urdf/crx10ia_l/crx10ia_l_sim.xacro (robot description, xacro)
@@ -2,4 +2,4 @@
 <robot name="crx10ia_l" xmlns:xacro="http://wiki.ros.org/xacro">
   <xacro:include filename="$(find crx_description)/urdf/crx10ia_l/crx10ia_l.urdf.xacro"/>
-  <xacro:crx10ia_l use_mock_hardware="false"/>
+  <xacro:crx10ia_l use_mock_hardware="true"/>
 </robot>
