Commit message: galileo : working on real robot and paametrized sim and real

File: urdf/crx10ia_l/crx10ia_l.xacro (robot description, xacro)
@@ -1,5 +1,9 @@
 <?xml version="1.0"?>
 <robot name="crx10ia_l" xmlns:xacro="http://wiki.ros.org/xacro">
+  <xacro:arg name="use_mock_hardware" default="true" />
+  <xacro:arg name="read_only" default="false" />
+  <xacro:arg name="robot_ip" default="192.168.150.2" />
+  <xacro:arg name="use_rmi" default="false" />
   <xacro:include filename="$(find crx_description)/urdf/crx10ia_l/crx10ia_l.urdf.xacro"/>
-  <xacro:crx10ia_l use_mock_hardware="false"/>
+  <xacro:crx10ia_l use_mock_hardware="$(arg use_mock_hardware)" robot_ip="$(arg robot_ip)" read_only="$(arg read_only)" use_rmi="$(arg use_rmi)"/>
 </robot>

File: urdf/crx20ia_l/crx20ia_l.urdf.xacro (robot description, xacro)
@@ -2,5 +2,5 @@
 <robot xmlns:xacro="http://wiki.ros.org/xacro">
   <xacro:macro name="crx20ia_l"
-               params="robot_ip:=192.168.150.2
+               params="robot_ip=192.168.150.2
                read_only=false
                use_rmi=false
@@ -58,15 +58,15 @@
     <link name="base_link">
       <visual>
-	<origin xyz="0 0 0" rpy="0 0 0"/>
-	<geometry>
-	  <mesh filename="package://crx_description/meshes/crx20ia_l/visual/base.stl" scale="0.001 0.001 0.001"/>
-	</geometry>
-	<material name="FANUC_Black"/>
-      </visual>
-      <collision>
-	<origin xyz="0 0 0" rpy="0 0 0"/>
-	<geometry>
-	  <mesh filename="package://crx_description/meshes/crx20ia_l/collision/base.stl" scale="0.001 0.001 0.001"/>
-	</geometry>
+      	<origin xyz="0 0 0" rpy="0 0 0"/>
+      	<geometry>
+      	  <mesh filename="package://crx_description/meshes/crx20ia_l/visual/base.stl" scale="0.001 0.001 0.001"/>
+      	</geometry>
+      	<material name="FANUC_Black"/>
+      </visual>
+      <collision>
+      	<origin xyz="0 0 0" rpy="0 0 0"/>
+      	<geometry>
+      	  <mesh filename="package://crx_description/meshes/crx20ia_l/collision/base.stl" scale="0.001 0.001 0.001"/>
+      	</geometry>
       </collision>
     </link>
@@ -74,14 +74,14 @@
       <visual>
         <origin xyz="0 0 ${mz_1 - l_base}" rpy="0 0 0"/>
-	<geometry>
-	  <mesh filename="package://crx_description/meshes/crx20ia_l/visual/j1.stl" scale="0.001 0.001 0.001"/>
-	</geometry>
-	<material name="FANUC_White"/>
+	       <geometry>
+	         <mesh filename="package://crx_description/meshes/crx20ia_l/visual/j1.stl" scale="0.001 0.001 0.001"/>
+    	   </geometry>
+        <material name="FANUC_White"/>
       </visual>
       <collision>
         <origin xyz="0 0 ${mz_1 - l_base}" rpy="0 0 0"/>
-	<geometry>
-	  <mesh filename="package://crx_description/meshes/crx20ia_l/collision/j1.stl" scale="0.001 0.001 0.001"/>
-	</geometry>
+    	  <geometry>
+          <mesh filename="package://crx_description/meshes/crx20ia_l/collision/j1.stl" scale="0.001 0.001 0.001"/>
+        </geometry>
       </collision>
     </link>
@@ -89,74 +89,74 @@
       <visual>
         <origin xyz="-${l_1} 0 ${mz_2 - l_base}" rpy="0 0 0"/>
-	<geometry>
-	  <mesh filename="package://crx_description/meshes/crx20ia_l/visual/j2.stl" scale="0.001 0.001 0.001"/>
-	</geometry>
-	<material name="FANUC_White"/>
+      	<geometry>
+          <mesh filename="package://crx_description/meshes/crx20ia_l/visual/j2.stl" scale="0.001 0.001 0.001"/>
+        </geometry>
+        <material name="FANUC_White"/>
       </visual>
       <collision>
         <origin xyz="-${l_1} 0 ${mz_2 - l_base}" rpy="0 0 0"/>
-	<geometry>
-	  <mesh filename="package://crx_description/meshes/crx20ia_l/collision/j2.stl" scale="0.001 0.001 0.001"/>
-	</geometry>
+        <geometry>
+          <mesh filename="package://crx_description/meshes/crx20ia_l/collision/j2.stl" scale="0.001 0.001 0.001"/>
+        </geometry>
       </collision>
     </link>
     <link name="J3_link">
       <visual>
-	<origin xyz="-${l_1} 0 ${mz_3 - l_base - l_2}" rpy="0 0 0"/>
-	<geometry>
-	  <mesh filename="package://crx_description/meshes/crx20ia_l/visual/j3.stl" scale="0.001 0.001 0.001"/>
-	</geometry>
-	<material name="FANUC_White"/>
-      </visual>
-      <collision>
-	<origin xyz="-${l_1} 0 ${mz_3 - l_base - l_2}" rpy="0 0 0"/>
-	<geometry>
-	  <mesh filename="package://crx_description/meshes/crx20ia_l/collision/j3.stl" scale="0.001 0.001 0.001"/>
-	</geometry>
+        <origin xyz="-${l_1} 0 ${mz_3 - l_base - l_2}" rpy="0 0 0"/>
+        <geometry>
+          <mesh filename="package://crx_description/meshes/crx20ia_l/visual/j3.stl" scale="0.001 0.001 0.001"/>
+        </geometry>
+        <material name="FANUC_White"/>
+      </visual>
+      <collision>
+        <origin xyz="-${l_1} 0 ${mz_3 - l_base - l_2}" rpy="0 0 0"/>
+        <geometry>
+          <mesh filename="package://crx_description/meshes/crx20ia_l/collision/j3.stl" scale="0.001 0.001 0.001"/>
+        </geometry>
       </collision>
     </link>
     <link name="J4_link">
       <visual>
-	<origin xyz="${mx_1 - l_1} 0 ${mz_3 - l_base - l_2 - l_3}" rpy="0 0 0"/>
-	<geometry>
-	  <mesh filename="package://crx_description/meshes/crx20ia_l/visual/j4.stl" scale="0.001 0.001 0.001"/>
-	</geometry>
-	<material name="FANUC_White"/>
-      </visual>
-      <collision>
-	<origin xyz="${mx_1 - l_1} 0 ${mz_3 - l_base - l_2 - l_3}" rpy="0 0 0"/>
-	<geometry>
-	  <mesh filename="package://crx_description/meshes/crx20ia_l/collision/j4.stl" scale="0.001 0.001 0.001"/>
-	</geometry>
+        <origin xyz="${mx_1 - l_1} 0 ${mz_3 - l_base - l_2 - l_3}" rpy="0 0 0"/>
+        <geometry>
+          <mesh filename="package://crx_description/meshes/crx20ia_l/visual/j4.stl" scale="0.001 0.001 0.001"/>
+        </geometry>
+        <material name="FANUC_White"/>
+      </visual>
+      <collision>
+        <origin xyz="${mx_1 - l_1} 0 ${mz_3 - l_base - l_2 - l_3}" rpy="0 0 0"/>
+        <geometry>
+          <mesh filename="package://crx_description/meshes/crx20ia_l/collision/j4.stl" scale="0.001 0.001 0.001"/>
+        </geometry>
       </collision>
     </link>
     <link name="J5_link">
       <visual>
-	<origin xyz="${mx_1 -l_1 - l_4} ${my_1} ${mz_3 - l_base - l_2 - l_3}" rpy="0 0 0"/>
-	<geometry>
-	  <mesh filename="package://crx_description/meshes/crx20ia_l/visual/j5.stl" scale="0.001 0.001 0.001"/>
-	</geometry>
-	<material name="FANUC_White"/>
-      </visual>
-      <collision>
-	<origin xyz="${mx_1 -l_1 - l_4} ${my_1} ${mz_3 - l_base - l_2 - l_3}" rpy="0 0 0"/>
-	<geometry>
-	  <mesh filename="package://crx_description/meshes/crx20ia_l/collision/j5.stl" scale="0.001 0.001 0.001"/>
-	</geometry>
+        <origin xyz="${mx_1 -l_1 - l_4} ${my_1} ${mz_3 - l_base - l_2 - l_3}" rpy="0 0 0"/>
+        <geometry>
+          <mesh filename="package://crx_description/meshes/crx20ia_l/visual/j5.stl" scale="0.001 0.001 0.001"/>
+        </geometry>
+        <material name="FANUC_White"/>
+      </visual>
+      <collision>
+        <origin xyz="${mx_1 -l_1 - l_4} ${my_1} ${mz_3 - l_base - l_2 - l_3}" rpy="0 0 0"/>
+        <geometry>
+          <mesh filename="package://crx_description/meshes/crx20ia_l/collision/j5.stl" scale="0.001 0.001 0.001"/>
+        </geometry>
       </collision>
     </link>
     <link name="J6_link">
       <visual>
-	<origin xyz="${mx_2 -l_1 - l_4} ${my_1 + l_5} ${mz_3 - l_base - l_2 - l_3}" rpy="0 0 0"/>
-	<geometry>
-	  <mesh filename="package://crx_description/meshes/crx20ia_l/visual/j6.stl" scale="0.001 0.001 0.001"/>
-	</geometry>
-	<material name="FANUC_Black"/>
-      </visual>
-      <collision>
-	<origin xyz="${mx_2 -l_1 - l_4} ${my_1 + l_5} ${mz_3 - l_base - l_2 - l_3}" rpy="0 0 0"/>
-	<geometry>
-	  <mesh filename="package://crx_description/meshes/crx20ia_l/collision/j6.stl" scale="0.001 0.001 0.001"/>
-	</geometry>
+        <origin xyz="${mx_2 -l_1 - l_4} ${my_1 + l_5} ${mz_3 - l_base - l_2 - l_3}" rpy="0 0 0"/>
+        <geometry>
+          <mesh filename="package://crx_description/meshes/crx20ia_l/visual/j6.stl" scale="0.001 0.001 0.001"/>
+        </geometry>
+        <material name="FANUC_Black"/>
+      </visual>
+      <collision>
+        <origin xyz="${mx_2 -l_1 - l_4} ${my_1 + l_5} ${mz_3 - l_base - l_2 - l_3}" rpy="0 0 0"/>
+        <geometry>
+          <mesh filename="package://crx_description/meshes/crx20ia_l/collision/j6.stl" scale="0.001 0.001 0.001"/>
+        </geometry>
       </collision>
     </link>

File: urdf/crx20ia_l/crx20ia_l.xacro (robot description, xacro)
@@ -1,7 +1,9 @@
 <?xml version="1.0"?>
 <robot name="crx20ia_l" xmlns:xacro="http://wiki.ros.org/xacro">
+  <xacro:arg name="use_mock_hardware" default="true" />
+  <xacro:arg name="read_only" default="false" />
+  <xacro:arg name="robot_ip" default="192.168.150.2" />
+  <xacro:arg name="use_rmi" default="false" />
   <xacro:include filename="$(find crx_description)/urdf/crx20ia_l/crx20ia_l.urdf.xacro"/>
-  <!-- <xacro:include filename="$(find crx_description)/crx20/urdf/crx20ia_l.ros2_control.xacro"/> -->
-  <xacro:crx20ia_l use_mock_hardware="false"/>
-  <!-- <xacro:crx20_ros2_control name="crx20"/> -->
+  <xacro:crx20ia_l use_mock_hardware="$(arg use_mock_hardware)" robot_ip="$(arg robot_ip)" read_only="$(arg read_only)" use_rmi="$(arg use_rmi)"/>
 </robot>

File: urdf/crx20ia_l/crx20ia_l_sim.xacro (robot description, xacro)
@@ -1,7 +1,8 @@
 <?xml version="1.0"?>
 <robot name="crx20ia_l" xmlns:xacro="http://wiki.ros.org/xacro">
+  <xacro:arg name="use_mock_hardware" default="true" />
   <xacro:include filename="$(find crx_description)/urdf/crx20ia_l/crx20ia_l.urdf.xacro"/>
   <!-- <xacro:include filename="$(find crx_description)/crx20/urdf/crx20ia_l.ros2_control.xacro"/> -->
-  <xacro:crx20ia_l use_mock_hardware="true"/>
+  <xacro:crx20ia_l use_mock_hardware="$(arg use_mock_hardware)"/>
   <!-- <xacro:crx20_ros2_control name="crx20"/> -->
 </robot>
