Commit message: galileo : fixed all descriptions

File: urdf/crx10ia/crx10ia.urdf.xacro (robot description, xacro)
@@ -1,8 +1,15 @@
 <?xml version="1.0"?>
 <robot xmlns:xacro="http://wiki.ros.org/xacro">
-  <xacro:macro name="crx10ia" params="use_mock_hardware:=false">
-  <xacro:arg name="use_mock_hardware" default="false"/>
+  <xacro:macro name="crx10ia"
+               params="robot_ip='10.11.31.121'
+               read_only='false'
+               use_rmi='false'
+               use_mock_hardware=false">
   <xacro:include filename="$(find crx_description)/urdf/crx.ros2_control.xacro"/>
-  <xacro:crx_ros2_control name="crx10" use_mock_hardware="$(arg use_mock_hardware)"/>
+  <xacro:crx_ros2_control name="crx10"
+                          use_mock_hardware="${use_mock_hardware}"
+                          robot_ip="${robot_ip}"
+                          read_only="${read_only}"
+                          use_rmi="${use_rmi}" />
     <material name="FANUC_Black">
       <color rgba="0 0 0 1.0"/>

File: urdf/crx10ia/crx10ia.xacro (robot description, xacro)
@@ -1,5 +1,9 @@
 <?xml version="1.0"?>
 <robot name="crx10ia" xmlns:xacro="http://wiki.ros.org/xacro">
+  <xacro:arg name="use_mock_hardware" default="true" />
+  <xacro:arg name="read_only" default="false" />
+  <xacro:arg name="robot_ip" default="192.168.150.2" />
+  <xacro:arg name="use_rmi" default="false" />
   <xacro:include filename="$(find crx_description)/urdf/crx10ia/crx10ia.urdf.xacro"/>
-  <xacro:crx10ia/>
+  <xacro:crx10ia use_mock_hardware="$(arg use_mock_hardware)" robot_ip="$(arg robot_ip)" read_only="$(arg read_only)" use_rmi="$(arg use_rmi)"/>
 </robot>

File: urdf/crx10ia_l/crx10ia_l.urdf.xacro (robot description, xacro)
@@ -31,10 +31,10 @@
     <xacro:property name="l_5" value="0.150"/>
     <xacro:property name="l_6" value="0.160"/>
-    <xacro:property name="j1_v" value="80"/>
-    <xacro:property name="j2_v" value="80"/>
-    <xacro:property name="j3_v" value="120"/>
-    <xacro:property name="j4_v" value="112.5"/>
-    <xacro:property name="j5_v" value="90"/>
-    <xacro:property name="j6_v" value="112.5"/>
+    <xacro:property name="j1_v" value="120"/>
+    <xacro:property name="j2_v" value="120"/>
+    <xacro:property name="j3_v" value="180"/>
+    <xacro:property name="j4_v" value="180"/>
+    <xacro:property name="j5_v" value="180"/>
+    <xacro:property name="j6_v" value="180"/>
     <xacro:property name="j1_u" value="179.9"/>
     <xacro:property name="j2_u" value="179.9"/>

File: urdf/crx25ia_l/crx25ia_l.urdf.xacro (robot description, xacro)
@@ -2,18 +2,14 @@
 <robot xmlns:xacro="http://wiki.ros.org/xacro">
   <xacro:macro name="crx25ia_l"
-               params="robot_ip:=10.11.31.101
-               use_rmi:=false
-               read_only:=false
-               use_mock_hardware:=false">
-  <xacro:arg name="use_mock_hardware" default="false"/>
-  <xacro:arg name="robot_ip" default="10.11.31.111"/>
-  <xacro:arg name="read_only" default="false"/>
-  <xacro:arg name="use_rmi" default="false"/>
-  <xacro:include filename="$(find crx_description)/urdf/crx.ros2_control.xacro"/>
-  <xacro:crx_ros2_control name="crx25"
-                          use_mock_hardware="$(arg use_mock_hardware)"
-                          robot_ip="$(arg robot_ip)"
-                          read_only="$(arg read_only)"
-                          use_rmi="$(arg use_rmi)"/>
+               params="robot_ip='10.11.31.121'
+               read_only='false'
+               use_rmi='false'
+               use_mock_hardware=false">
+    <xacro:include filename="$(find crx_description)/urdf/crx.ros2_control.xacro"/>
+    <xacro:crx_ros2_control name="crx25"
+                            use_mock_hardware="${use_mock_hardware}"
+                            robot_ip="${robot_ip}"
+                            read_only="${read_only}"
+                            use_rmi="${use_rmi}" />
     <material name="FANUC_Black">
       <color rgba="0 0 0 1.0"/>

File: urdf/crx25ia_l/crx25ia_l.xacro (robot description, xacro)
@@ -1,7 +1,9 @@
 <?xml version="1.0"?>
 <robot name="crx25ia_l" xmlns:xacro="http://wiki.ros.org/xacro">
+  <xacro:arg name="use_mock_hardware" default="true" />
+  <xacro:arg name="read_only" default="false" />
+  <xacro:arg name="robot_ip" default="192.168.150.2" />
+  <xacro:arg name="use_rmi" default="false" />
   <xacro:include filename="$(find crx_description)/urdf/crx25ia_l/crx25ia_l.urdf.xacro"/>
-  <!-- <xacro:include filename="$(find crx_description)/crx25/urdf/crx25ia_l.ros2_control.xacro"/> -->
-  <xacro:crx25ia_l/>
-  <!-- <xacro:crx25_ros2_control name="crx25"/> -->
+  <xacro:crx25ia_l use_mock_hardware="$(arg use_mock_hardware)" robot_ip="$(arg robot_ip)" read_only="$(arg read_only)" use_rmi="$(arg use_rmi)"/>
 </robot>

File: urdf/crx5ia/crx5ia.urdf.xacro (robot description, xacro)
@@ -1,8 +1,15 @@
 <?xml version="1.0"?>
 <robot xmlns:xacro="http://wiki.ros.org/xacro">
-  <xacro:macro name="crx5" params="use_mock_hardware:=false">
-  <xacro:arg name="use_mock_hardware" default="false"/>
+  <xacro:macro name="crx5ia"
+                params="robot_ip='10.11.31.121'
+                read_only='false'
+                use_rmi='false'
+                use_mock_hardware=false">
   <xacro:include filename="$(find crx_description)/urdf/crx.ros2_control.xacro"/>
-  <xacro:crx_ros2_control name="crx5" use_mock_hardware="$(arg use_mock_hardware)"/>
+  <xacro:crx_ros2_control name="crx5"
+                          use_mock_hardware="${use_mock_hardware}"
+                          robot_ip="${robot_ip}"
+                          read_only="${read_only}"
+                          use_rmi="${use_rmi}" />
     <material name="FANUC_Black">
       <color rgba="0 0 0 1.0"/>

File: urdf/crx5ia/crx5ia.xacro (robot description, xacro)
@@ -1,5 +1,9 @@
 <?xml version="1.0"?>
-<robot name="crx5" xmlns:xacro="http://wiki.ros.org/xacro">
+<robot name="crx5ia" xmlns:xacro="http://wiki.ros.org/xacro">
+  <xacro:arg name="use_mock_hardware" default="true" />
+  <xacro:arg name="read_only" default="false" />
+  <xacro:arg name="robot_ip" default="192.168.150.2" />
+  <xacro:arg name="use_rmi" default="false" />
   <xacro:include filename="$(find crx_description)/urdf/crx5ia/crx5ia.urdf.xacro"/>
-  <xacro:crx5/>
+  <xacro:crx5ia use_mock_hardware="$(arg use_mock_hardware)" robot_ip="$(arg robot_ip)" read_only="$(arg read_only)" use_rmi="$(arg use_rmi)"/>
 </robot>
